File: wireless-temperaure-sensor.kicad_pcb (KiCad board)
At the start: 2 copper layers, 18 parts, among them J1 Programmer, U1 stm32l010f4, U2 NRF24L01_Breakout, U3 MCP9808_MSOP

Commit message: Finalised first draft version of PCB
Parts:
- C4: moved to B.Cu
- moved BT1 29.3 mm to (106.7, 97.8)
- moved C1 23.9 mm to (110.7, 115.6), turned to 0 degrees
Routing:
- net VDD: track 38.9 -> 164.8 mm, vias 0 -> 3
- net /MOSI: track 50.8 -> 49.1 mm
- net /SPI_SCK: track 44.9 -> 44.0 mm
- net GND: track 0.00 -> 0.65 mm, vias 0 -> 2
- net /MISO: track 44.2 -> 43.7 mm
- added copper zone on B.Cu, net GND
- added copper zone on F.Cu, net GND
Other:
- board outline added: 45.1 x 55.9 mm
